Commit message: Obtaining robot arm

File: rei_dsl/rei_dsl/temp.urdf (robot description, URDF)
Before this commit: robot basic_robot, 8 links, 7 joints
Links:
- removed link caster_wheel_caster_root
- removed link caster_wheel_caster_wheel_link
- removed link caster_wheel_tire_link
- removed link left_wheel_wheel_axle
- removed link left_wheel_wheel_link
- removed link right_wheel_wheel_axle
- removed link right_wheel_wheel_link
- added link arm_link; collision cylinder length=0.6 radius=0.1; visual cylinder length=0.6 radius=0.1
- added link shoulder_link; collision cylinder length=0.1 radius=0.15; visual cylinder length=0.1 radius=0.15
- added link wrist_link1; collision cylinder length=0.1 radius=0.1; visual cylinder length=0.1 radius=0.1
- added link wrist_link2; collision cylinder length=0.1 radius=0.1; visual cylinder length=0.1 radius=0.1
- added link wrist_link3; collision cylinder length=0.1 radius=0.1; visual cylinder length=0.3 radius=0.1
- link base_link: mass None -> 10.0; geometry collision cylinder length=0.3 radius=0.2; visual cylinder length=0.3 radius=0.2
Joints:
- removed joint caster_wheel_jnt_caster_root
- removed joint caster_wheel_jnt_caster_tire
- removed joint jnt_caster_wheel_connect
- removed joint jnt_left_wheel_connect
- removed joint jnt_right_wheel_connect
- removed joint left_wheel_jnt_left_wheel
- removed joint right_wheel_jnt_left_wheel
- added joint jnt_arm_wrist: type revolute, parent arm_link, child wrist_link1, origin xyz=0.0 0.0 0.6 rpy=0.0 0.0 0.0, axis 1 0 0, limit lower=-2.0943951023931953 upper=2.0943951023931953
- added joint jnt_base_shoulder: type revolute, parent base_link, child shoulder_link, origin xyz=0.0 0.0 0.1 rpy=0.0 0.0 0.0, axis 0 0 1, limit lower=-3.141592653589793 upper=3.141592653589793
- added joint jnt_shoulder_arm: type revolute, parent shoulder_link, child arm_link, origin xyz=0.0 0.0 0.15 rpy=0.0 0.0 0.0, axis 1 0 0, limit lower=-2.0943951023931953 upper=2.0943951023931953
- added joint jnt_wrist1_wrist2: type revolute, parent wrist_link1, child wrist_link2, origin xyz=0.0 0.0 0.075 rpy=0.0 0.0 0.0, axis 0 0 1, limit lower=-2.0943951023931953 upper=2.0943951023931953
- added joint jnt_wrist2_wrist3: type revolute, parent wrist_link2, child wrist_link3, origin xyz=0.0 0.0 0.075 rpy=0.0 0.0 0.0, axis 1 0 0, limit lower=-2.0943951023931953 upper=2.0943951023931953

Commit message: Cyberdisc added

File: rei_dsl/rei_dsl/temp.urdf (robot description, URDF)
Before this commit: robot basic_anthropomorph, 6 links, 5 joints
Links:
- removed link arm_link
- removed link shoulder_link
- removed link wrist_link1
- removed link wrist_link2
- removed link wrist_link3
- added link motor_0_motor_axle; collision cylinder length=0.07 radius=0.005; visual cylinder length=0.07 radius=0.005
- added link motor_0_motor_root; collision box size=0.08 0.04 0.03; visual box size=0.08 0.04 0.03
- added link motor_0_wheel_link; collision cylinder length=0.02 radius=0.04; visual cylinder length=0.02 radius=0.04
- added link motor_1_motor_axle; collision cylinder length=0.07 radius=0.005; visual cylinder length=0.07 radius=0.005
- added link motor_1_motor_root; collision box size=0.08 0.04 0.03; visual box size=0.08 0.04 0.03
- added link motor_1_wheel_link; collision cylinder length=0.02 radius=0.04; visual cylinder length=0.02 radius=0.04
- added link motor_2_motor_axle; collision cylinder length=0.07 radius=0.005; visual cylinder length=0.07 radius=0.005
- added link motor_2_motor_root; collision box size=0.08 0.04 0.03; visual box size=0.08 0.04 0.03
- added link motor_2_wheel_link; collision cylinder length=0.02 radius=0.04; visual cylinder length=0.02 radius=0.04
- added link motor_3_motor_axle; collision cylinder length=0.07 radius=0.005; visual cylinder length=0.07 radius=0.005
- added link motor_3_motor_root; collision box size=0.08 0.04 0.03; visual box size=0.08 0.04 0.03
- added link motor_3_wheel_link; collision cylinder length=0.02 radius=0.04; visual cylinder length=0.02 radius=0.04
- link base_link: mass 10.0 -> None; geometry collision cylinder length=0.05 radius=0.25; visual cylinder length=0.05 radius=0.25
Joints:
- removed joint jnt_arm_wrist
- removed joint jnt_base_shoulder
- removed joint jnt_shoulder_arm
- removed joint jnt_wrist1_wrist2
- removed joint jnt_wrist2_wrist3
- added joint jnt_motor_0_connect: type fixed, parent base_link, child motor_0_motor_root, origin xyz=0.1 0.1 0.0 rpy=0.0 0.0 1.5707963267948966
- added joint jnt_motor_1_connect: type fixed, parent base_link, child motor_1_motor_root, origin xyz=-0.1 0.1 0.0 rpy=0.0 0.0 1.5707963267948966
- added joint jnt_motor_2_connect: type fixed, parent base_link, child motor_2_motor_root, origin xyz=-0.1 -0.1 0.0 rpy=0.0 0.0 -1.5707963267948966
- added joint jnt_motor_3_connect: type fixed, parent base_link, child motor_3_motor_root, origin xyz=0.1 -0.1 0.0 rpy=0.0 0.0 -1.5707963267948966
- added joint motor_0_jnt_motor: type fixed, parent motor_0_motor_root, child motor_0_motor_axle, origin xyz=0.04 0.0 0.0 rpy=0.0 1.5707963267948966 0.0
- added joint motor_0_jnt_motor_wheel: type continuous, parent motor_0_motor_axle, child motor_0_wheel_link, origin xyz=0.0 0.0 0.0 rpy=0.0 0.0 0.0, axis 0 0 1
- added joint motor_1_jnt_motor: type fixed, parent motor_1_motor_root, child motor_1_motor_axle, origin xyz=0.04 0.0 0.0 rpy=0.0 1.5707963267948966 0.0
- added joint motor_1_jnt_motor_wheel: type continuous, parent motor_1_motor_axle, child motor_1_wheel_link, origin xyz=0.0 0.0 0.0 rpy=0.0 0.0 0.0, axis 0 0 1
- added joint motor_2_jnt_motor: type fixed, parent motor_2_motor_root, child motor_2_motor_axle, origin xyz=0.04 0.0 0.0 rpy=0.0 1.5707963267948966 0.0
- added joint motor_2_jnt_motor_wheel: type continuous, parent motor_2_motor_axle, child motor_2_wheel_link, origin xyz=0.0 0.0 0.0 rpy=0.0 0.0 0.0, axis 0 0 1
- added joint motor_3_jnt_motor: type fixed, parent motor_3_motor_root, child motor_3_motor_axle, origin xyz=0.04 0.0 0.0 rpy=0.0 1.5707963267948966 0.0
- added joint motor_3_jnt_motor_wheel: type continuous, parent motor_3_motor_axle, child motor_3_wheel_link, origin xyz=0.0 0.0 0.0 rpy=0.0 0.0 0.0, axis 0 0 1
